Commit message: [Update] InverseKinematics done

File: src/px_robot/urdf/px_collision.urdf (robot description, URDF)
Before this commit: robot px_robot, 7 links, 6 joints
Joints:
- joint joint_1: origin xyz=0.0 0.0 0.09 rpy=0.0 0.0 0.0 -> xyz=0.0 0.0 0.05 rpy=0.0 0.0 0.0
- joint joint_3: origin xyz=0.05 0.1065 0 rpy=0.0 0.0 -1.5707 -> xyz=0.037 0.103 0 rpy=0.0 0.0 -1.5707
- joint joint_4: origin xyz=0.0 0.1065 0 rpy=0.0 0.0 0.0 -> xyz=0.0 0.098 0 rpy=0.0 0.0 0.0
- joint tcp: origin xyz=0.0 0.092 0 rpy=-1.5707 0.0 0.0 -> xyz=0.0 0.0114 0 rpy=-1.5707 0.0 0.0
